Commit message: feat: 更新至EDULITE-A3模型，添加夹爪控制
主要更新:
- 替换URDF为EDULITE-A3模型
- 更新所有3D mesh文件
- 更新关节限位参数
- 配置电机方向 (L1/L3/L5=-1, L2/L4/L6=+1)
- 添加夹爪控制 (ID=7, 方向键上下控制±0.4Nm)
- 完成惯性参数标定 (inertia_params.yaml)
- 更新README文档

File: ros2_ws/src/rs_a3_web_ui/static/urdf/rs_a3.urdf (robot description, URDF)
Before this commit: robot RS-A3, 9 links, 8 joints
Links:
- link l1_link_urdf_asm: mass 0.140779 -> 0.146738; geometry collision mesh filename=package://rs_a3_description/meshes/part_8.stl; collision mesh filename=package://rs_a3_description/meshes/part_9.stl
- link l1_urdf_urdf_asm: mass 0.410786 -> 0.465144; geometry collision mesh filename=package://rs_a3_description/meshes/part_10.stl; collision mesh filename=package://rs_a3_description/meshes/rs00_l1.stl
- link l2_l3_urdf_asm: mass 0.83477 -> 0.946534
- link l3_lnik_urdf_asm: mass 0.197637 -> 0.406558; geometry collision mesh filename=package://rs_a3_description/meshes/small_arm_left.stl; collision mesh filename=package://rs_a3_description/meshes/small_arm_right.stl
- link l4_l5_urdf_asm: mass 0.46061 -> 0.44692
- link l5_l6_urdf_asm: mass 0.53126 -> 0.5317; geometry collision mesh filename=package://rs_a3_description/meshes/hand_r.stl; collision mesh filename=package://rs_a3_description/meshes/manifold_solid_brep_39_1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
- link part_9: mass 0.0179604 -> 0.0179457; geometry collision mesh filename=package://rs_a3_description/meshes/part_9__2.stl; visual mesh filename=package://rs_a3_description/meshes/part_9__2.stl
Joints:
- joint L1_joint: limit lower=-6.28 upper=6.28 effort=14 velocity=33 -> lower=-2.79253 upper=2.79253 effort=14 velocity=33; origin xyz=0 0 0.0054 rpy=0 0 0 -> xyz=0 0 0.006 rpy=0 0 0
- joint L2_joint: limit lower=-6.28 upper=6.28 effort=14 velocity=33 -> lower=0 upper=3.66519 effort=14 velocity=33; origin xyz=-0.0176846 0 0.0606 rpy=1.5708 0 0 -> xyz=-0.01 -0.0006 0.064 rpy=1.5708 0 0
- joint L3_joint: limit lower=-6.28 upper=6.28 effort=14 velocity=33 -> lower=-4.01426 upper=0 effort=14 velocity=33; origin xyz=0.19 0 0 rpy=0 0 0 -> xyz=0.19 0 0.0518 rpy=0 0 0
- joint L4_joint: limit lower=-6.28 upper=6.28 effort=5.5 velocity=50 -> lower=-1.5708 upper=1.5708 effort=5.5 velocity=50; origin xyz=-0.15 0.06 0 rpy=0 0 0 -> xyz=-0.185 0.064 -0.0518 rpy=0 0 0
- joint L5_joint: limit lower=-6.28 upper=6.28 effort=5.5 velocity=50 -> lower=-1.5708 upper=1.5708 effort=5.5 velocity=50
- joint L6_joint: limit lower=-6.28 upper=6.28 effort=5.5 velocity=50 -> lower=-1.5708 upper=1.5708 effort=5.5 velocity=50; origin xyz=0.00805 0 0.038 rpy=1.5708 0 -1.5708 -> xyz=0.00805 0 0.038 rpy=-1.5708 0 -1.5708
- joint end_effector_joint: origin xyz=0 0 0.074 rpy=0 0 0 -> xyz=0 0 -0.074 rpy=0 0 0

File: rs_a3_description/urdf/rs_a3.urdf.xacro (robot description, xacro)
@@ -1,4 +1,5 @@
 <?xml version="1.0" ?>
 <!-- RS-A3 6-DOF Robot Arm URDF with ros2_control support -->
+<!-- Updated from EDULITE-A3 model -->
 <robot name="RS-A3" xmlns:xacro="http://www.ros.org/wiki/xacro">
   <!-- Arguments -->
@@ -30,4 +31,7 @@
     <color rgba="0.980392 0.713725 0.00392157 1"/>
   </material>
+  <material name="green">
+    <color rgba="0.372549 0.654902 0.239216 1"/>
+  </material>
   <!-- Base link (world) -->
   <link name="base_link"/>
@@ -40,12 +44,27 @@
   <link name="l1_urdf_urdf_asm">
     <inertial>
-      <origin xyz="-0.000473642 -3.66697e-05 -0.0209915" rpy="0 0 0"/>
-      <mass value="0.410786"/>
-      <inertia ixx="0.000243951" ixy="-2.931e-09" ixz="-2.71862e-06"
-               iyy="0.000233462" iyz="5.03989e-07" izz="0.000256472"/>
+      <origin xyz="-2.68984e-10 1.48294e-05 -0.0220571" rpy="0 0 0"/>
+      <mass value="0.465144"/>
+      <inertia ixx="0.00032748" ixy="-1.33894e-08" ixz="-1.85358e-12"
+               iyy="0.000321793" iyz="-2.46949e-07" izz="0.000362426"/>
     </inertial>
+    <!-- Part part_10 -->
     <visual>
       <origin xyz="0 0 0" rpy="0 0 0"/>
       <geometry>
+        <mesh filename="package://rs_a3_description/meshes/part_10.stl"/>
+      </geometry>
+      <material name="green"/>
+    </visual>
+    <collision>
+      <origin xyz="0 0 0" rpy="0 0 0"/>
+      <geometry>
+        <mesh filename="package://rs_a3_description/meshes/part_10.stl"/>
+      </geometry>
+    </collision>
+    <!-- Part rs00_l1 -->
+    <visual>
+      <origin xyz="0 0 0" rpy="0 0 0"/>
+      <geometry>
         <mesh filename="package://rs_a3_description/meshes/rs00_l1.stl"/>
       </geometry>
@@ -56,17 +75,4 @@
       <geometry>
         <mesh filename="package://rs_a3_description/meshes/rs00_l1.stl"/>
-      </geometry>
-    </collision>
-    <visual>
-      <origin xyz="0 0 0" rpy="0 0 0"/>
-      <geometry>
-        <mesh filename="package://rs_a3_description/meshes/l1_base.stl"/>
-      </geometry>
-      <material name="gray"/>
-    </visual>
-    <collision>
-      <origin xyz="0 0 0" rpy="0 0 0"/>
-      <geometry>
-        <mesh filename="package://rs_a3_description/meshes/l1_base.stl"/>
       </geometry>
     </collision>
@@ -75,46 +81,35 @@
   <link name="l1_link_urdf_asm">
     <inertial>
-      <origin xyz="-0.00670261 -0.000377334 0.0342178" rpy="0 0 0"/>
-      <mass value="0.140779"/>
-      <inertia ixx="0.000189723" ixy="-1.61467e-06" ixz="1.97828e-05"
-               iyy="0.000112632" iyz="3.73644e-06" izz="0.00016217"/>
+      <origin xyz="-0.00202103 -0.00162495 0.0394318" rpy="0 0 0"/>
+      <mass value="0.146738"/>
+      <inertia ixx="0.000221617" ixy="-1.44161e-06" ixz="1.46922e-05"
+               iyy="0.000129193" iyz="4.22954e-06" izz="0.000175411"/>
     </inertial>
-    <visual>
-      <origin xyz="0 0 -0.0054" rpy="0 0 0"/>
-      <geometry>
-        <mesh filename="package://rs_a3_description/meshes/l1_link_stop.stl"/>
-      </geometry>
-      <material name="light_blue"/>
-    </visual>
-    <collision>
-      <origin xyz="0 0 -0.0054" rpy="0 0 0"/>
-      <geometry>
-        <mesh filename="package://rs_a3_description/meshes/l1_link_stop.stl"/>
-      </geometry>
-    </collision>
-    <visual>
-      <origin xyz="0 0 -0.0054" rpy="0 0 0"/>
-      <geometry>
-        <mesh filename="package://rs_a3_description/meshes/l1_link_drv.stl"/>
-      </geometry>
-      <material name="light_blue"/>
-    </visual>
-    <collision>
-      <origin xyz="0 0 -0.0054" rpy="0 0 0"/>
-      <geometry>
-        <mesh filename="package://rs_a3_description/meshes/l1_link_drv.stl"/>
-      </geometry>
-    </collision>
-    <visual>
-      <origin xyz="0 0 -0.0054" rpy="0 0 0"/>
-      <geometry>
-        <mesh filename="package://rs_a3_description/meshes/l2_stop.stl"/>
-      </geometry>
-      <material name="orange"/>
-    </visual>
-    <collision>
-      <origin xyz="0 0 -0.0054" rpy="0 0 0"/>
-      <geometry>
-        <mesh filename="package://rs_a3_description/meshes/l2_stop.stl"/>
+    <!-- Part part_8 -->
+    <visual>
+      <origin xyz="0 0 -0.006" rpy="0 0 0"/>
+      <geometry>
+        <mesh filename="package://rs_a3_description/meshes/part_8.stl"/>
+      </geometry>
+      <material name="yellow"/>
+    </visual>
+    <collision>
+      <origin xyz="0 0 -0.006" rpy="0 0 0"/>
+      <geometry>
+        <mesh filename="package://rs_a3_description/meshes/part_8.stl"/>
+      </geometry>
+    </collision>
+    <!-- Part part_9 -->
+    <visual>
+      <origin xyz="0 0 -0.006" rpy="0 0 0"/>
+      <geometry>
+        <mesh filename="package://rs_a3_description/meshes/part_9.stl"/>
+      </geometry>
+      <material name="yellow"/>
+    </visual>
+    <collision>
+      <origin xyz="0 0 -0.006" rpy="0 0 0"/>
+      <geometry>
+        <mesh filename="package://rs_a3_description/meshes/part_9.stl"/>
       </geometry>
     </collision>
@@ -123,11 +118,12 @@
   <link name="l2_l3_urdf_asm">
     <inertial>
-      <origin xyz="0.095 -3.5032e-07 -0.000569607" rpy="0 0 0"/>
-      <mass value="0.83477"/>
-      <inertia ixx="0.000411892" ixy="-2.68928e-08" ixz="8.18489e-11"
-               iyy="0.0070909" iyz="-4.27746e-09" izz="0.00710532"/>
+      <origin xyz="0.0949994 -1.38262e-06 -0.00108795" rpy="0 0 0"/>
+      <mass value="0.946534"/>
+      <inertia ixx="0.000493341" ixy="6.92125e-07" ixz="-1.27006e-08"
+               iyy="0.00767087" iyz="2.73309e-09" izz="0.0076934"/>
     </inertial>
-    <visual>
-      <origin xyz="0.0176846 -0.066 0.0005" rpy="-1.5708 0 0"/>
+    <!-- Part mainlink_back -->
+    <visual>
+      <origin xyz="0.01 -0.07 -0.0001" rpy="-1.5708 0 0"/>
       <geometry>
         <mesh filename="package://rs_a3_description/meshes/mainlink_back.stl"/>
@@ -136,11 +132,12 @@
     </visual>
     <collision>
-      <origin xyz="0.0176846 -0.066 0.0005" rpy="-1.5708 0 0"/>
+      <origin xyz="0.01 -0.07 -0.0001" rpy="-1.5708 0 0"/>
       <geometry>
         <mesh filename="package://rs_a3_description/meshes/mainlink_back.stl"/>
       </geometry>
     </collision>
-    <visual>
-      <origin xyz="0.0176846 -0.066 0.0005" rpy="-1.5708 0 0"/>
+    <!-- Part 6705 -->
+    <visual>
+      <origin xyz="0.01 -0.07 -0.0001" rpy="-1.5708 0 0"/>
       <geometry>
         <mesh filename="package://rs_a3_description/meshes/6705.stl"/>
@@ -149,11 +146,12 @@
     </visual>
     <collision>
-      <origin xyz="0.0176846 -0.066 0.0005" rpy="-1.5708 0 0"/>
+      <origin xyz="0.01 -0.07 -0.0001" rpy="-1.5708 0 0"/>
       <geometry>
         <mesh filename="package://rs_a3_description/meshes/6705.stl"/>
       </geometry>
     </collision>
-    <visual>
-      <origin xyz="0.0176846 -0.066 0" rpy="-1.5708 0 0"/>
+    <!-- Part rs00_l2 -->
+    <visual>
+      <origin xyz="0.01 -0.07 -0.0006" rpy="-1.5708 0 0"/>
       <geometry>
         <mesh filename="package://rs_a3_description/meshes/rs00_l2.stl"/>
@@ -162,11 +160,12 @@
     </visual>
     <collision>
-      <origin xyz="0.0176846 -0.066 0" rpy="-1.5708 0 0"/>
+      <origin xyz="0.01 -0.07 -0.0006" rpy="-1.5708 0 0"/>
       <geometry>
         <mesh filename="package://rs_a3_description/meshes/rs00_l2.stl"/>
       </geometry>
     </collision>
-    <visual>
-      <origin xyz="0.0176846 -0.066 0" rpy="-1.5708 0 0"/>
+    <!-- Part mainlink_motor -->
+    <visual>
+      <origin xyz="0.01 -0.07 -0.0006" rpy="-1.5708 0 0"/>
       <geometry>
         <mesh filename="package://rs_a3_description/meshes/mainlink_motor.stl"/>
@@ -175,11 +174,12 @@
     </visual>
     <collision>
-      <origin xyz="0.0176846 -0.066 0" rpy="-1.5708 0 0"/>
+      <origin xyz="0.01 -0.07 -0.0006" rpy="-1.5708 0 0"/>
       <geometry>
         <mesh filename="package://rs_a3_description/meshes/mainlink_motor.stl"/>
       </geometry>
     </collision>
-    <visual>
-      <origin xyz="0.0176846 -0.066 0.0005" rpy="-1.5708 0 0"/>
+    <!-- Part 6705_2 -->
+    <visual>
+      <origin xyz="0.01 -0.07 -0.0001" rpy="-1.5708 0 0"/>
       <geometry>
         <mesh filename="package://rs_a3_description/meshes/6705__2.stl"/>
@@ -188,11 +188,12 @@
     </visual>
     <collision>
-      <origin xyz="0.0176846 -0.066 0.0005" rpy="-1.5708 0 0"/>
+      <origin xyz="0.01 -0.07 -0.0001" rpy="-1.5708 0 0"/>
       <geometry>
         <mesh filename="package://rs_a3_description/meshes/6705__2.stl"/>
       </geometry>
     </collision>
-    <visual>
-      <origin xyz="0.0176846 -0.066 0" rpy="-1.5708 0 0"/>
+    <!-- Part rs00_l3 -->
+    <visual>
+      <origin xyz="0.01 -0.07 -0.0006" rpy="-1.5708 0 0"/>
       <geometry>
         <mesh filename="package://rs_a3_description/meshes/rs00_l3.stl"/>
@@ -201,5 +202,5 @@
     </visual>
     <collision>
-      <origin xyz="0.0176846 -0.066 0" rpy="-1.5708 0 0"/>
+      <origin xyz="0.01 -0.07 -0.0006" rpy="-1.5708 0 0"/>
       <geometry>
         <mesh filename="package://rs_a3_description/meshes/rs00_l3.stl"/>
@@ -210,33 +211,35 @@
   <link name="l3_lnik_urdf_asm">
     <inertial>
-      <origin xyz="-0.055871 0.0492802 0.0027754" rpy="0 0 0"/>
-      <mass value="0.197637"/>
-      <inertia ixx="0.000241191" ixy="0.000108757" ixz="-7.09292e-06"
-               iyy="0.000663739" iyz="6.85788e-06" izz="0.000641507"/>
+      <origin xyz="-0.0693243 0.0530595 -0.0510805" rpy="0 0 0"/>
+      <mass value="0.406558"/>
+      <inertia ixx="0.000554036" ixy="0.000274809" ixz="4.74842e-06"
+               iyy="0.00189339" iyz="7.79959e-06" izz="0.00192037"/>
     </inertial>
-    <visual>
-      <origin xyz="-0.172315 -0.066 0" rpy="-1.5708 0 0"/>
-      <geometry>
-        <mesh filename="package://rs_a3_description/meshes/l4_link_back.stl"/>
-      </geometry>
-      <material name="dark_gray"/>
-    </visual>
-    <collision>
-      <origin xyz="-0.172315 -0.066 0" rpy="-1.5708 0 0"/>
-      <geometry>
-        <mesh filename="package://rs_a3_description/meshes/l4_link_back.stl"/>
-      </geometry>
-    </collision>
-    <visual>
-      <origin xyz="-0.172315 -0.066 0" rpy="-1.5708 0 0"/>
-      <geometry>
-        <mesh filename="package://rs_a3_description/meshes/l4_link_drv.stl"/>
-      </geometry>
-      <material name="dark_gray"/>
-    </visual>
-    <collision>
-      <origin xyz="-0.172315 -0.066 0" rpy="-1.5708 0 0"/>
-      <geometry>
-        <mesh filename="package://rs_a3_description/meshes/l4_link_drv.stl"/>
+    <!-- Part small_arm_right -->
+    <visual>
+      <origin xyz="-0.18 -0.07 -0.0518" rpy="-1.5708 0 0"/>
+      <geometry>
+        <mesh filename="package://rs_a3_description/meshes/small_arm_right.stl"/>
+      </geometry>
+      <material name="orange"/>
+    </visual>
+    <collision>
+      <origin xyz="-0.18 -0.07 -0.0518" rpy="-1.5708 0 0"/>
+      <geometry>
+        <mesh filename="package://rs_a3_description/meshes/small_arm_right.stl"/>
+      </geometry>
+    </collision>
+    <!-- Part small_arm_left -->
+    <visual>
+      <origin xyz="-0.18 -0.07 -0.0518" rpy="-1.5708 0 0"/>
+      <geometry>
+        <mesh filename="package://rs_a3_description/meshes/small_arm_left.stl"/>
+      </geometry>
+      <material name="orange"/>
+    </visual>
+    <collision>
+      <origin xyz="-0.18 -0.07 -0.0518" rpy="-1.5708 0 0"/>
+      <geometry>
+        <mesh filename="package://rs_a3_description/meshes/small_arm_left.stl"/>
       </geometry>
     </collision>
@@ -245,11 +248,12 @@
   <link name="l4_l5_urdf_asm">
     <inertial>
-      <origin xyz="-0.0242557 0.0305328 -0.000278918" rpy="0 0 0"/>
-      <mass value="0.46061"/>
-      <inertia ixx="0.000570996" ixy="0.000329291" ixz="3.22513e-06"
-               iyy="0.000412235" iyz="-4.05021e-06" izz="0.000827873"/>
+      <origin xyz="-0.0241077 0.0297756 -0.000254349" rpy="0 0 0"/>
+      <mass value="0.44692"/>
+      <inertia ixx="0.000543249" ixy="0.000320527" ixz="2.88671e-06"
+               iyy="0.00040341" iyz="-3.57587e-06" izz="0.000797799"/>
     </inertial>
-    <visual>
-      <origin xyz="-0.0223154 -0.126 0" rpy="-1.5708 0 0"/>
+    <!-- Part rs05_l5 -->
+    <visual>
+      <origin xyz="0.005 -0.134 0" rpy="-1.5708 0 0"/>
       <geometry>
         <mesh filename="package://rs_a3_description/meshes/rs05_l5.stl"/>
@@ -258,37 +262,54 @@
     </visual>
     <collision>
-      <origin xyz="-0.0223154 -0.126 0" rpy="-1.5708 0 0"/>
+      <origin xyz="0.005 -0.134 0" rpy="-1.5708 0 0"/>
       <geometry>
         <mesh filename="package://rs_a3_description/meshes/rs05_l5.stl"/>
       </geometry>
     </collision>
-    <visual>
-      <origin xyz="-0.0223154 -0.126 0" rpy="-1.5708 0 0"/>
+    <!-- Part l5_shake -->
+    <visual>
+      <origin xyz="0.005 -0.134 0" rpy="-1.5708 0 0"/>
+      <geometry>
+        <mesh filename="package://rs_a3_description/meshes/l5_shake.stl"/>
+      </geometry>
+      <material name="light_blue"/>
+    </visual>
+    <collision>
+      <origin xyz="0.005 -0.134 0" rpy="-1.5708 0 0"/>
+      <geometry>
+        <mesh filename="package://rs_a3_description/meshes/l5_shake.stl"/>
+      </geometry>
+    </collision>
+    <!-- Part l4_l5_link_back -->
+    <visual>
+      <origin xyz="0.005 -0.134 0" rpy="-1.5708 0 0"/>
       <geometry>
         <mesh filename="package://rs_a3_description/meshes/l4_l5_link_back.stl"/>
       </geometry>
-      <material name="white"/>
-    </visual>
-    <collision>
-      <origin xyz="-0.0223154 -0.126 0" rpy="-1.5708 0 0"/>
+      <material name="orange"/>
+    </visual>
+    <collision>
+      <origin xyz="0.005 -0.134 0" rpy="-1.5708 0 0"/>
       <geometry>
         <mesh filename="package://rs_a3_description/meshes/l4_l5_link_back.stl"/>
       </geometry>
     </collision>
-    <visual>
-      <origin xyz="-0.0223154 -0.126 0" rpy="-1.5708 0 0"/>
-      <geometry>
-        <mesh filename="package://rs_a3_description/meshes/l5_shake.stl"/>
-      </geometry>
-      <material name="light_blue"/>
-    </visual>
-    <collision>
-      <origin xyz="-0.0223154 -0.126 0" rpy="-1.5708 0 0"/>
-      <geometry>
-        <mesh filename="package://rs_a3_description/meshes/l5_shake.stl"/>
-      </geometry>
-    </collision>
-    <visual>
-      <origin xyz="-0.0223154 -0.126 0" rpy="-1.5708 0 0"/>
+    <!-- Part rs05_l4 -->
+    <visual>
+      <origin xyz="0.005 -0.134 0" rpy="-1.5708 0 0"/>
+      <geometry>
+        <mesh filename="package://rs_a3_description/meshes/rs05_l4.stl"/>
+      </geometry>
+      <material name="white"/>
+    </visual>
+    <collision>
+      <origin xyz="0.005 -0.134 0" rpy="-1.5708 0 0"/>
+      <geometry>
+        <mesh filename="package://rs_a3_description/meshes/rs05_l4.stl"/>
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
File: rs_a3_description/urdf/rs_a3_ros2_control.xacro (robot description, xacro)
@@ -26,5 +26,5 @@
           <param name="gravity_feedforward_ratio">0.5</param>  <!-- 50%重力补偿比例 -->
           <!-- 零力矩模式参数 -->
-          <param name="zero_torque_kd">0.1</param>  <!-- 零力矩模式阻尼系数 -->
+          <param name="zero_torque_kd">0.03</param>  <!-- 零力矩模式阻尼系数 -->
           <!-- Pinocchio 动力学模型配置 -->
           <!-- 注意：需要设置 URDF 文件的绝对路径 -->
@@ -96,6 +96,6 @@
         <param name="direction">1.0</param>
         <command_interface name="position">
-          <param name="min">-3.14159</param>
-          <param name="max">3.14159</param>
+          <param name="min">0</param>
+          <param name="max">3.66519</param>
         </command_interface>
         <command_interface name="velocity">
@@ -118,6 +118,6 @@
         <param name="direction">-1.0</param>
         <command_interface name="position">
-          <param name="min">-3.14159</param>
-          <param name="max">3.14159</param>
+          <param name="min">-4.01426</param>
+          <param name="max">0</param>
         </command_interface>
         <command_interface name="velocity">
@@ -140,6 +140,6 @@
         <param name="direction">1.0</param>
         <command_interface name="position">
-          <param name="min">-3.14159</param>
-          <param name="max">3.14159</param>
+          <param name="min">-1.5708</param>
+          <param name="max">1.5708</param>
         </command_interface>
         <command_interface name="velocity">
@@ -162,6 +162,6 @@
         <param name="direction">-1.0</param>
         <command_interface name="position">
-          <param name="min">-3.14159</param>
-          <param name="max">3.14159</param>
+          <param name="min">-1.5708</param>
+          <param name="max">1.5708</param>
         </command_interface>
         <command_interface name="velocity">
@@ -182,8 +182,8 @@
         <param name="motor_type">RS05</param>
         <param name="position_offset">0.0</param>
-        <param name="direction">-1.0</param>
-        <command_interface name="position">
-          <param name="min">-3.14159</param>
-          <param name="max">3.14159</param>
+        <param name="direction">1.0</param>
+        <command_interface name="position">
+          <param name="min">-1.5708</param>
+          <param name="max">1.5708</param>
         </command_interface>
         <command_interface name="velocity">
