Commit message: feat: 添加多机械臂控制支持
- 添加 URDF prefix 参数支持多机械臂命名空间
- 创建多臂配置文件 (multi_arm_config.yaml)
- 创建多臂控制器配置 (multi_arm_controllers.yaml)
- 创建多臂启动文件 (multi_arm_control.launch.py)
- 创建主从遥操作节点 (支持一对多、多对多映射)
- 创建主从配置文件 (master_slave_config.yaml)
- 添加多 CAN 接口配置脚本 (setup_multi_can.sh)
- 更新 README 添加多臂控制使用说明

File: rs_a3_description/urdf/rs_a3.urdf.xacro (robot description, xacro)
@@ -4,7 +4,10 @@
 <robot name="RS-A3" xmlns:xacro="http://www.ros.org/wiki/xacro">
   <!-- Arguments -->
+  <xacro:arg name="prefix" default=""/>
   <xacro:arg name="use_mock_hardware" default="false"/>
   <xacro:arg name="can_interface" default="can0"/>
   <xacro:arg name="host_can_id" default="253"/>
+  <!-- Properties for prefix -->
+  <xacro:property name="prefix" value="$(arg prefix)"/>
   <!-- Include ros2_control -->
   <xacro:include filename="$(find rs_a3_description)/urdf/rs_a3_ros2_control.xacro"/>
@@ -35,12 +38,12 @@
   </material>
   <!-- Base link (world) -->
-  <link name="base_link"/>
-  <joint name="base_to_l1" type="fixed">
-    <parent link="base_link"/>
-    <child link="l1_urdf_urdf_asm"/>
+  <link name="${prefix}base_link"/>
+  <joint name="${prefix}base_to_l1" type="fixed">
+    <parent link="${prefix}base_link"/>
+    <child link="${prefix}l1_urdf_urdf_asm"/>
     <origin xyz="0 0 0" rpy="0 0 0"/>
   </joint>
   <!-- Link l1_urdf_urdf_asm (Base) -->
-  <link name="l1_urdf_urdf_asm">
+  <link name="${prefix}l1_urdf_urdf_asm">
     <inertial>
       <origin xyz="-2.68984e-10 1.48294e-05 -0.0220571" rpy="0 0 0"/>
@@ -79,5 +82,5 @@
   </link>
   <!-- Link l1_link_urdf_asm -->
-  <link name="l1_link_urdf_asm">
+  <link name="${prefix}l1_link_urdf_asm">
     <inertial>
       <origin xyz="-0.00202103 -0.00162495 0.0394318" rpy="0 0 0"/>
@@ -116,5 +119,5 @@
   </link>
   <!-- Link l2_l3_urdf_asm -->
-  <link name="l2_l3_urdf_asm">
+  <link name="${prefix}l2_l3_urdf_asm">
     <inertial>
       <origin xyz="0.0949994 -1.38262e-06 -0.00108795" rpy="0 0 0"/>
@@ -209,5 +212,5 @@
   </link>
   <!-- Link l3_lnik_urdf_asm -->
-  <link name="l3_lnik_urdf_asm">
+  <link name="${prefix}l3_lnik_urdf_asm">
     <inertial>
       <origin xyz="-0.0693243 0.0530595 -0.0510805" rpy="0 0 0"/>
@@ -246,5 +249,5 @@
   </link>
   <!-- Link l4_l5_urdf_asm -->
-  <link name="l4_l5_urdf_asm">
+  <link name="${prefix}l4_l5_urdf_asm">
     <inertial>
       <origin xyz="-0.0241077 0.0297756 -0.000254349" rpy="0 0 0"/>
@@ -325,5 +328,5 @@
   </link>
   <!-- Link part_9 -->
-  <link name="part_9">
+  <link name="${prefix}part_9">
     <inertial>
       <origin xyz="0.00409255 0 0.0175119" rpy="0 0 0"/>
@@ -348,5 +351,5 @@
   </link>
   <!-- Link l5_l6_urdf_asm (End Effector) -->
-  <link name="l5_l6_urdf_asm">
+  <link name="${prefix}l5_l6_urdf_asm">
     <inertial>
       <origin xyz="-1.16996e-05 0.000627615 -0.0701883" rpy="0 0 0"/>
@@ -553,11 +556,11 @@
   </link>
   <!-- End Effector link -->
-  <link name="end_effector"/>
+  <link name="${prefix}end_effector"/>
   <!-- Joints -->
   <!-- Joint L1 (RS00 Motor 1) -->
-  <joint name="L1_joint" type="revolute">
+  <joint name="${prefix}L1_joint" type="revolute">
     <origin xyz="0 0 0.006" rpy="0 0 0"/>
-    <parent link="l1_urdf_urdf_asm"/>
-    <child link="l1_link_urdf_asm"/>
+    <parent link="${prefix}l1_urdf_urdf_asm"/>
+    <child link="${prefix}l1_link_urdf_asm"/>
     <axis xyz="0 0 1"/>
     <limit effort="14" velocity="33" lower="-2.79253" upper="2.79253"/>
@@ -565,8 +568,8 @@
   </joint>
   <!-- Joint L2 (RS00 Motor 2) -->
-  <joint name="L2_joint" type="revolute">
+  <joint name="${prefix}L2_joint" type="revolute">
     <origin xyz="-0.01 -0.0006 0.064" rpy="1.5708 0 0"/>
-    <parent link="l1_link_urdf_asm"/>
-    <child link="l2_l3_urdf_asm"/>
+    <parent link="${prefix}l1_link_urdf_asm"/>
+    <child link="${prefix}l2_l3_urdf_asm"/>
     <axis xyz="0 0 1"/>
     <limit effort="14" velocity="33" lower="0" upper="3.66519"/>
@@ -574,8 +577,8 @@
   </joint>
   <!-- Joint L3 (RS00 Motor 3) -->
-  <joint name="L3_joint" type="revolute">
+  <joint name="${prefix}L3_joint" type="revolute">
     <origin xyz="0.19 0 0.0518" rpy="0 0 0"/>
-    <parent link="l2_l3_urdf_asm"/>
-    <child link="l3_lnik_urdf_asm"/>
+    <parent link="${prefix}l2_l3_urdf_asm"/>
+    <child link="${prefix}l3_lnik_urdf_asm"/>
     <axis xyz="0 0 1"/>
     <limit effort="14" velocity="33" lower="-4.01426" upper="0"/>
@@ -583,8 +586,8 @@
   </joint>
   <!-- Joint L4 (RS05 Motor 4) -->
-  <joint name="L4_joint" type="revolute">
+  <joint name="${prefix}L4_joint" type="revolute">
     <origin xyz="-0.185 0.064 -0.0518" rpy="0 0 0"/>
-    <parent link="l3_lnik_urdf_asm"/>
-    <child link="l4_l5_urdf_asm"/>
+    <parent link="${prefix}l3_lnik_urdf_asm"/>
+    <child link="${prefix}l4_l5_urdf_asm"/>
     <axis xyz="0 0 1"/>
     <limit effort="5.5" velocity="50" lower="-1.5708" upper="1.5708"/>
@@ -592,8 +595,8 @@
   </joint>
   <!-- Joint L5 (RS05 Motor 5) -->
-  <joint name="L5_joint" type="revolute">
+  <joint name="${prefix}L5_joint" type="revolute">
     <origin xyz="-0.0492 0.038 0" rpy="1.5708 0 0"/>
-    <parent link="l4_l5_urdf_asm"/>
-    <child link="part_9"/>
+    <parent link="${prefix}l4_l5_urdf_asm"/>
+    <child link="${prefix}part_9"/>
     <axis xyz="0 0 1"/>
     <limit effort="5.5" velocity="50" lower="-1.5708" upper="1.5708"/>
@@ -601,8 +604,8 @@
   </joint>
   <!-- Joint L6 (RS05 Motor 6) -->
-  <joint name="L6_joint" type="revolute">
+  <joint name="${prefix}L6_joint" type="revolute">
     <origin xyz="0.00805 0 0.038" rpy="-1.5708 0 -1.5708"/>
-    <parent link="part_9"/>
-    <child link="l5_l6_urdf_asm"/>
+    <parent link="${prefix}part_9"/>
+    <child link="${prefix}l5_l6_urdf_asm"/>
     <axis xyz="0 0 1"/>
     <limit effort="5.5" velocity="50" lower="-1.5708" upper="1.5708"/>
@@ -610,11 +613,12 @@
   </joint>
   <!-- End Effector joint -->
-  <joint name="end_effector_joint" type="fixed">
+  <joint name="${prefix}end_effector_joint" type="fixed">
     <origin xyz="0 0 -0.074" rpy="0 0 0"/>
-    <parent link="l5_l6_urdf_asm"/>
-    <child link="end_effector"/>
+    <parent link="${prefix}l5_l6_urdf_asm"/>
+    <child link="${prefix}end_effector"/>
   </joint>
   <!-- ros2_control interface -->
   <xacro:rs_a3_ros2_control
+    prefix="$(arg prefix)"
     use_mock_hardware="$(arg use_mock_hardware)"
     can_interface="$(arg can_interface)"

File: rs_a3_description/urdf/rs_a3_ros2_control.xacro (robot description, xacro)
@@ -2,6 +2,6 @@
 <!-- RS-A3 ros2_control configuration -->
 <robot xmlns:xacro="http://www.ros.org/wiki/xacro">
-  <xacro:macro name="rs_a3_ros2_control" params="use_mock_hardware can_interface host_can_id">
-    <ros2_control name="RsA3System" type="system">
+  <xacro:macro name="rs_a3_ros2_control" params="prefix use_mock_hardware can_interface host_can_id">
+    <ros2_control name="${prefix}RsA3System" type="system">
       <hardware>
         <xacro:if value="${use_mock_hardware}">
@@ -82,5 +82,5 @@
       </hardware>
       <!-- Joint L1 - RS00 Motor 1 -->
-      <joint name="L1_joint">
+      <joint name="${prefix}L1_joint">
         <param name="motor_id">1</param>
         <param name="motor_type">RS00</param>
@@ -104,5 +104,5 @@
       </joint>
       <!-- Joint L2 - RS00 Motor 2 -->
-      <joint name="L2_joint">
+      <joint name="${prefix}L2_joint">
         <param name="motor_id">2</param>
         <param name="motor_type">RS00</param>
@@ -126,5 +126,5 @@
       </joint>
       <!-- Joint L3 - RS00 Motor 3 -->
-      <joint name="L3_joint">
+      <joint name="${prefix}L3_joint">
         <param name="motor_id">3</param>
         <param name="motor_type">RS00</param>
@@ -148,5 +148,5 @@
       </joint>
       <!-- Joint L4 - RS05 Motor 4 -->
-      <joint name="L4_joint">
+      <joint name="${prefix}L4_joint">
         <param name="motor_id">4</param>
         <param name="motor_type">RS05</param>
@@ -170,5 +170,5 @@
       </joint>
       <!-- Joint L5 - RS05 Motor 5 -->
-      <joint name="L5_joint">
+      <joint name="${prefix}L5_joint">
         <param name="motor_id">5</param>
         <param name="motor_type">RS05</param>
@@ -192,5 +192,5 @@
       </joint>
       <!-- Joint L6 - RS05 Motor 6 -->
-      <joint name="L6_joint">
+      <joint name="${prefix}L6_joint">
         <param name="motor_id">6</param>
         <param name="motor_type">RS05</param>
