Commit message: feat: 添加视觉抓取、主从遥操作增强、EDULITE-A3模型和多项改进
- 添加 rs_a3_vision 视觉抓取包（相机节点、物体检测、手眼标定、视觉伺服）
- 添加 rs_a3_grasp_gui 抓取GUI包
- 添加 EDULITE-A3 原始URDF和mesh模型文件
- 增强主从遥操作节点（多臂支持、配置优化）
- 更新多臂控制launch和配置（multi_arm_config、controllers）
- 更新URDF xacro和ros2_control配置
- 优化硬件接口（零力矩模式服务路径更新）
- 精简惯性参数标定脚本
- 添加arm2独立惯性参数配置
- 添加重力标定工具和分析脚本
- 添加遥操作和测试脚本
- 更新README文档
- 移除已跟踪的__pycache__文件

Co-authored-by: Cursor <cursoragent@cursor.com>

File: rs_a3_description/urdf/rs_a3.urdf.xacro (robot description, xacro)
@@ -4,10 +4,7 @@
 <robot name="RS-A3" xmlns:xacro="http://www.ros.org/wiki/xacro">
   <!-- Arguments -->
-  <xacro:arg name="prefix" default=""/>
   <xacro:arg name="use_mock_hardware" default="false"/>
   <xacro:arg name="can_interface" default="can0"/>
   <xacro:arg name="host_can_id" default="253"/>
-  <!-- Properties for prefix -->
-  <xacro:property name="prefix" value="$(arg prefix)"/>
   <!-- Include ros2_control -->
   <xacro:include filename="$(find rs_a3_description)/urdf/rs_a3_ros2_control.xacro"/>
@@ -38,12 +35,12 @@
   </material>
   <!-- Base link (world) -->
-  <link name="${prefix}base_link"/>
-  <joint name="${prefix}base_to_l1" type="fixed">
-    <parent link="${prefix}base_link"/>
-    <child link="${prefix}l1_urdf_urdf_asm"/>
+  <link name="base_link"/>
+  <joint name="base_to_l1" type="fixed">
+    <parent link="base_link"/>
+    <child link="l1_urdf_urdf_asm"/>
     <origin xyz="0 0 0" rpy="0 0 0"/>
   </joint>
   <!-- Link l1_urdf_urdf_asm (Base) -->
-  <link name="${prefix}l1_urdf_urdf_asm">
+  <link name="l1_urdf_urdf_asm">
     <inertial>
       <origin xyz="-2.68984e-10 1.48294e-05 -0.0220571" rpy="0 0 0"/>
@@ -82,5 +79,5 @@
   </link>
   <!-- Link l1_link_urdf_asm -->
-  <link name="${prefix}l1_link_urdf_asm">
+  <link name="l1_link_urdf_asm">
     <inertial>
       <origin xyz="-0.00202103 -0.00162495 0.0394318" rpy="0 0 0"/>
@@ -119,5 +116,5 @@
   </link>
   <!-- Link l2_l3_urdf_asm -->
-  <link name="${prefix}l2_l3_urdf_asm">
+  <link name="l2_l3_urdf_asm">
     <inertial>
       <origin xyz="0.0949994 -1.38262e-06 -0.00108795" rpy="0 0 0"/>
@@ -212,5 +209,5 @@
   </link>
   <!-- Link l3_lnik_urdf_asm -->
-  <link name="${prefix}l3_lnik_urdf_asm">
+  <link name="l3_lnik_urdf_asm">
     <inertial>
       <origin xyz="-0.0693243 0.0530595 -0.0510805" rpy="0 0 0"/>
@@ -249,5 +246,5 @@
   </link>
   <!-- Link l4_l5_urdf_asm -->
-  <link name="${prefix}l4_l5_urdf_asm">
+  <link name="l4_l5_urdf_asm">
     <inertial>
       <origin xyz="-0.0241077 0.0297756 -0.000254349" rpy="0 0 0"/>
@@ -328,5 +325,5 @@
   </link>
   <!-- Link part_9 -->
-  <link name="${prefix}part_9">
+  <link name="part_9">
     <inertial>
       <origin xyz="0.00409255 0 0.0175119" rpy="0 0 0"/>
@@ -351,5 +348,5 @@
   </link>
   <!-- Link l5_l6_urdf_asm (End Effector) -->
-  <link name="${prefix}l5_l6_urdf_asm">
+  <link name="l5_l6_urdf_asm">
     <inertial>
       <origin xyz="-1.16996e-05 0.000627615 -0.0701883" rpy="0 0 0"/>
@@ -556,11 +553,11 @@
   </link>
   <!-- End Effector link -->
-  <link name="${prefix}end_effector"/>
+  <link name="end_effector"/>
   <!-- Joints -->
   <!-- Joint L1 (RS00 Motor 1) -->
-  <joint name="${prefix}L1_joint" type="revolute">
+  <joint name="L1_joint" type="revolute">
     <origin xyz="0 0 0.006" rpy="0 0 0"/>
-    <parent link="${prefix}l1_urdf_urdf_asm"/>
-    <child link="${prefix}l1_link_urdf_asm"/>
+    <parent link="l1_urdf_urdf_asm"/>
+    <child link="l1_link_urdf_asm"/>
     <axis xyz="0 0 1"/>
     <limit effort="14" velocity="33" lower="-2.79253" upper="2.79253"/>
@@ -568,8 +565,8 @@
   </joint>
   <!-- Joint L2 (RS00 Motor 2) -->
-  <joint name="${prefix}L2_joint" type="revolute">
+  <joint name="L2_joint" type="revolute">
     <origin xyz="-0.01 -0.0006 0.064" rpy="1.5708 0 0"/>
-    <parent link="${prefix}l1_link_urdf_asm"/>
-    <child link="${prefix}l2_l3_urdf_asm"/>
+    <parent link="l1_link_urdf_asm"/>
+    <child link="l2_l3_urdf_asm"/>
     <axis xyz="0 0 1"/>
     <limit effort="14" velocity="33" lower="0" upper="3.66519"/>
@@ -577,8 +574,8 @@
   </joint>
   <!-- Joint L3 (RS00 Motor 3) -->
-  <joint name="${prefix}L3_joint" type="revolute">
+  <joint name="L3_joint" type="revolute">
     <origin xyz="0.19 0 0.0518" rpy="0 0 0"/>
-    <parent link="${prefix}l2_l3_urdf_asm"/>
-    <child link="${prefix}l3_lnik_urdf_asm"/>
+    <parent link="l2_l3_urdf_asm"/>
+    <child link="l3_lnik_urdf_asm"/>
     <axis xyz="0 0 1"/>
     <limit effort="14" velocity="33" lower="-4.01426" upper="0"/>
@@ -586,8 +583,8 @@
   </joint>
   <!-- Joint L4 (RS05 Motor 4) -->
-  <joint name="${prefix}L4_joint" type="revolute">
+  <joint name="L4_joint" type="revolute">
     <origin xyz="-0.185 0.064 -0.0518" rpy="0 0 0"/>
-    <parent link="${prefix}l3_lnik_urdf_asm"/>
-    <child link="${prefix}l4_l5_urdf_asm"/>
+    <parent link="l3_lnik_urdf_asm"/>
+    <child link="l4_l5_urdf_asm"/>
     <axis xyz="0 0 1"/>
     <limit effort="5.5" velocity="50" lower="-1.5708" upper="1.5708"/>
@@ -595,8 +592,8 @@
   </joint>
   <!-- Joint L5 (RS05 Motor 5) -->
-  <joint name="${prefix}L5_joint" type="revolute">
+  <joint name="L5_joint" type="revolute">
     <origin xyz="-0.0492 0.038 0" rpy="1.5708 0 0"/>
-    <parent link="${prefix}l4_l5_urdf_asm"/>
-    <child link="${prefix}part_9"/>
+    <parent link="l4_l5_urdf_asm"/>
+    <child link="part_9"/>
     <axis xyz="0 0 1"/>
     <limit effort="5.5" velocity="50" lower="-1.5708" upper="1.5708"/>
@@ -604,8 +601,8 @@
   </joint>
   <!-- Joint L6 (RS05 Motor 6) -->
-  <joint name="${prefix}L6_joint" type="revolute">
+  <joint name="L6_joint" type="revolute">
     <origin xyz="0.00805 0 0.038" rpy="-1.5708 0 -1.5708"/>
-    <parent link="${prefix}part_9"/>
-    <child link="${prefix}l5_l6_urdf_asm"/>
+    <parent link="part_9"/>
+    <child link="l5_l6_urdf_asm"/>
     <axis xyz="0 0 1"/>
     <limit effort="5.5" velocity="50" lower="-1.5708" upper="1.5708"/>
@@ -613,12 +610,11 @@
   </joint>
   <!-- End Effector joint -->
-  <joint name="${prefix}end_effector_joint" type="fixed">
+  <joint name="end_effector_joint" type="fixed">
     <origin xyz="0 0 -0.074" rpy="0 0 0"/>
-    <parent link="${prefix}l5_l6_urdf_asm"/>
-    <child link="${prefix}end_effector"/>
+    <parent link="l5_l6_urdf_asm"/>
+    <child link="end_effector"/>
   </joint>
   <!-- ros2_control interface -->
   <xacro:rs_a3_ros2_control
-    prefix="$(arg prefix)"
     use_mock_hardware="$(arg use_mock_hardware)"
     can_interface="$(arg can_interface)"

File: rs_a3_description/urdf/rs_a3_ros2_control.xacro (robot description, xacro)
@@ -2,6 +2,6 @@
 <!-- RS-A3 ros2_control configuration -->
 <robot xmlns:xacro="http://www.ros.org/wiki/xacro">
-  <xacro:macro name="rs_a3_ros2_control" params="prefix use_mock_hardware can_interface host_can_id">
-    <ros2_control name="${prefix}RsA3System" type="system">
+  <xacro:macro name="rs_a3_ros2_control" params="use_mock_hardware can_interface host_can_id">
+    <ros2_control name="RsA3System" type="system">
       <hardware>
         <xacro:if value="${use_mock_hardware}">
@@ -26,19 +26,5 @@
           <param name="gravity_feedforward_ratio">0.5</param>  <!-- 50%重力补偿比例 -->
           <!-- 零力矩模式参数 -->
-          <param name="zero_torque_kd">0.3</param>  <!-- 零力矩模式默认阻尼系数 -->
-          <!-- 零力矩模式关节独立 Kp（通常为0，可微调提供轻微位置保持） -->
-          <param name="zero_torque_kp_L1">0.0</param>
-          <param name="zero_torque_kp_L2">0.0</param>
-          <param name="zero_torque_kp_L3">0.0</param>
-          <param name="zero_torque_kp_L4">0.0</param>
-          <param name="zero_torque_kp_L5">0.0</param>
-          <param name="zero_torque_kp_L6">0.0</param>
-          <!-- 零力矩模式关节独立 Kd（RS00大电机需要更高阻尼） -->
-          <param name="zero_torque_kd_L1">0.17</param>
-          <param name="zero_torque_kd_L2">0.35</param>  <!-- 大臂，高阻尼 -->
-          <param name="zero_torque_kd_L3">0.40</param>  <!-- 小臂 -->
-          <param name="zero_torque_kd_L4">0.05</param>
-          <param name="zero_torque_kd_L5">0.05</param>
-          <param name="zero_torque_kd_L6">0.05</param>
+          <param name="zero_torque_kd">0.3</param>  <!-- 零力矩模式阻尼系数 -->
           <!-- Pinocchio 动力学模型配置 -->
           <!-- 注意：需要设置 URDF 文件的绝对路径 -->
@@ -82,5 +68,5 @@
       </hardware>
       <!-- Joint L1 - RS00 Motor 1 -->
-      <joint name="${prefix}L1_joint">
+      <joint name="L1_joint">
         <param name="motor_id">1</param>
         <param name="motor_type">RS00</param>
@@ -104,5 +90,5 @@
       </joint>
       <!-- Joint L2 - RS00 Motor 2 -->
-      <joint name="${prefix}L2_joint">
+      <joint name="L2_joint">
         <param name="motor_id">2</param>
         <param name="motor_type">RS00</param>
@@ -126,5 +112,5 @@
       </joint>
       <!-- Joint L3 - RS00 Motor 3 -->
-      <joint name="${prefix}L3_joint">
+      <joint name="L3_joint">
         <param name="motor_id">3</param>
         <param name="motor_type">RS00</param>
@@ -148,5 +134,5 @@
       </joint>
       <!-- Joint L4 - RS05 Motor 4 -->
-      <joint name="${prefix}L4_joint">
+      <joint name="L4_joint">
         <param name="motor_id">4</param>
         <param name="motor_type">RS05</param>
@@ -170,5 +156,5 @@
       </joint>
       <!-- Joint L5 - RS05 Motor 5 -->
-      <joint name="${prefix}L5_joint">
+      <joint name="L5_joint">
         <param name="motor_id">5</param>
         <param name="motor_type">RS05</param>
@@ -192,5 +178,5 @@
       </joint>
       <!-- Joint L6 - RS05 Motor 6 -->
-      <joint name="${prefix}L6_joint">
+      <joint name="L6_joint">
         <param name="motor_id">6</param>
         <param name="motor_type">RS05</param>
