Commit message: feat: 全面重命名 RS-A3 → EL-A3，RS05 电机型号 → EL05
- 将所有 RS05 电机型号引用更改为 EL05（代码、配置、文档）
- 更新 EL05 扭矩映射范围：±5.5Nm → ±6Nm
- 重命名所有 rs_a3/RS-A3/RS_A3 目录和文件为 el_a3/EL-A3/EL_A3
- 重命名 rs05*.stl/part 网格文件为 el05*
- 更新所有文件中的路径引用和包名称

Co-authored-by: Cursor <cursoragent@cursor.com>

File: EDULITE-A3/EDULITE-A3.urdf (robot description, URDF)
Before this commit: robot EDULITE-A3, 7 links, 6 joints
Links:
- link l4_l5_urdf_asm: geometry collision mesh filename=package://edulite_a3_description/meshes/el05_l4.stl; collision mesh filename=package://edulite_a3_description/meshes/el05_l5.stl
- link l5_l6_urdf_asm: geometry collision mesh filename=package://edulite_a3_description/meshes/el05.stl; collision mesh filename=package://edulite_a3_description/meshes/el05.stl
