Commit message: feat: 添加 EL-A3 Python SDK、控制参数调优、SDK API 文档
- 新增 el_a3_sdk 完整 Python SDK（CAN 直连 + ROS Control 双模式）
  - ELA3Interface: CAN 直连控制接口
  - ELA3ROSInterface: ROS2 Control 集成接口
  - ArmManager: 单例多臂管理器
  - ELA3Kinematics: Pinocchio 运动学/动力学
  - 轨迹规划: S-curve 七段式 + 三次样条
  - Web SDK Bridge: REST API + WebSocket 命令桥接
- 控制参数调优（抑制手柄控制抖动）
  - 全局 Kp: 80→55, Kd: 4→4.5
  - 腕关节 L4-L6 独立 PD: Kp=30, Kd=2
  - 重力补偿比例: 50%→85%
  - 速度前馈 EMA 滤波: alpha 0.08/0.10→0.18/0.18
  - 手柄关节平滑: alpha 0.35→0.25
- 新增 ZeroTorqueController 独立控制器插件
- 支持 wrist_motor_type 参数 (EL05/RS05 可切换)
- 添加 SDK API 协议说明文档 (1277 行)
- 添加 rs_a3_hardware 兼容符号链接和测试脚本

Made-with: Cursor

File: el_a3_description/urdf/el_a3.urdf.xacro (robot description, xacro)
@@ -7,4 +7,8 @@
   <xacro:arg name="can_interface" default="can0"/>
   <xacro:arg name="host_can_id" default="253"/>
+  <xacro:arg name="wrist_motor_type" default="EL05"/>
+  <!-- Wrist motor parameters (EL05: 6Nm, RS05: 5.5Nm) -->
+  <xacro:property name="wrist_motor_type" value="$(arg wrist_motor_type)"/>
+  <xacro:property name="wrist_effort" value="${5.5 if wrist_motor_type == 'RS05' else 6.0}"/>
   <!-- Include ros2_control -->
   <xacro:include filename="$(find el_a3_description)/urdf/el_a3_ros2_control.xacro"/>
@@ -582,5 +586,5 @@
     <dynamics damping="0.1" friction="0.1"/>
   </joint>
-  <!-- Joint L4 (EL05 Motor 4) -->
+  <!-- Joint L4 (${wrist_motor_type} Motor 4) -->
   <joint name="L4_joint" type="revolute">
     <origin xyz="-0.185 0.064 -0.0518" rpy="0 0 0"/>
@@ -588,8 +592,8 @@
     <child link="l4_l5_urdf_asm"/>
     <axis xyz="0 0 1"/>
-    <limit effort="6.0" velocity="50" lower="-1.5708" upper="1.5708"/>
+    <limit effort="${wrist_effort}" velocity="50" lower="-1.5708" upper="1.5708"/>
     <dynamics damping="0.05" friction="0.05"/>
   </joint>
-  <!-- Joint L5 (EL05 Motor 5) -->
+  <!-- Joint L5 (${wrist_motor_type} Motor 5) -->
   <joint name="L5_joint" type="revolute">
     <origin xyz="-0.0492 0.038 0" rpy="1.5708 0 0"/>
@@ -597,8 +601,8 @@
     <child link="part_9"/>
     <axis xyz="0 0 1"/>
-    <limit effort="6.0" velocity="50" lower="-1.5708" upper="1.5708"/>
+    <limit effort="${wrist_effort}" velocity="50" lower="-1.5708" upper="1.5708"/>
     <dynamics damping="0.05" friction="0.05"/>
   </joint>
-  <!-- Joint L6 (EL05 Motor 6) -->
+  <!-- Joint L6 (${wrist_motor_type} Motor 6) -->
   <joint name="L6_joint" type="revolute">
     <origin xyz="0.00805 0 0.038" rpy="-1.5708 0 -1.5708"/>
@@ -606,8 +610,8 @@
     <child link="l5_l6_urdf_asm"/>
     <axis xyz="0 0 1"/>
-    <limit effort="6.0" velocity="50" lower="-1.5708" upper="1.5708"/>
+    <limit effort="${wrist_effort}" velocity="50" lower="-1.5708" upper="1.5708"/>
     <dynamics damping="0.05" friction="0.05"/>
   </joint>
-  <!-- End Effector joint -->
+  <!-- End Effector joint (fixed to last arm link, defines TCP for MoveIt planning) -->
   <joint name="end_effector_joint" type="fixed">
     <origin xyz="0 0 -0.074" rpy="0 0 0"/>
@@ -615,8 +619,25 @@
     <child link="end_effector"/>
   </joint>
+  <!-- Joint L7 (${wrist_motor_type} Motor 7 - Gripper, separate kinematic branch) -->
+  <joint name="L7_joint" type="revolute">
+    <origin xyz="0 0 -0.074" rpy="0 0 0"/>
+    <parent link="l5_l6_urdf_asm"/>
+    <child link="gripper_link"/>
+    <axis xyz="0 0 1"/>
+    <limit effort="${wrist_effort}" velocity="50" lower="-1.5708" upper="1.5708"/>
+    <dynamics damping="0.05" friction="0.05"/>
+  </joint>
+  <link name="gripper_link">
+    <inertial>
+      <mass value="0.05"/>
+      <origin xyz="0 0 0"/>
+      <inertia ixx="0.0001" ixy="0" ixz="0" iyy="0.0001" iyz="0" izz="0.0001"/>
+    </inertial>
+  </link>
   <!-- ros2_control interface -->
   <xacro:el_a3_ros2_control
     use_mock_hardware="$(arg use_mock_hardware)"
     can_interface="$(arg can_interface)"
-    host_can_id="$(arg host_can_id)"/>
+    host_can_id="$(arg host_can_id)"
+    wrist_motor_type="$(arg wrist_motor_type)"/>
 </robot>

File: el_a3_description/urdf/el_a3_ros2_control.xacro (robot description, xacro)
@@ -2,5 +2,8 @@
 <!-- EL-A3 ros2_control configuration -->
 <robot xmlns:xacro="http://www.ros.org/wiki/xacro">
-  <xacro:macro name="el_a3_ros2_control" params="use_mock_hardware can_interface host_can_id">
+  <xacro:macro name="el_a3_ros2_control" params="use_mock_hardware can_interface host_can_id wrist_motor_type">
+    <!-- Wrist motor effort limits based on motor type -->
+    <xacro:property name="wrist_effort_max" value="${5.5 if wrist_motor_type == 'RS05' else 6.0}"/>
+    <xacro:property name="wrist_effort_min" value="${-5.5 if wrist_motor_type == 'RS05' else -6.0}"/>
     <ros2_control name="RsA3System" type="system">
       <hardware>
@@ -13,6 +16,6 @@
           <param name="can_interface">${can_interface}</param>
           <param name="host_can_id">${host_can_id}</param>
-          <param name="position_kp">80.0</param>
-          <param name="position_kd">4.0</param>
+          <param name="position_kp">55.0</param>
+          <param name="position_kd">4.5</param>
           <param name="velocity_limit">10.0</param>
           <!-- S-curve trajectory planning parameters -->
@@ -23,6 +26,6 @@
           <!-- Fallback smoothing filter parameters (used when S-curve is disabled) -->
           <param name="smoothing_alpha">0.2</param>     <!-- Low-pass filter coefficient -->
-          <!-- Gravity compensation feedforward parameters (50% gravity as feedforward torque) -->
-          <param name="gravity_feedforward_ratio">0.5</param>  <!-- 50% gravity compensation ratio -->
+          <!-- Gravity compensation feedforward parameters (100% gravity as feedforward torque, matching zero-torque mode) -->
+          <param name="gravity_feedforward_ratio">0.85</param>  <!-- 85% gravity compensation ratio, avoid over-compensation oscillation -->
           <!-- Zero-torque mode parameters -->
           <param name="zero_torque_kd">0.3</param>  <!-- Zero-torque mode damping coefficient -->
@@ -133,65 +136,93 @@
         <state_interface name="effort"/>
       </joint>
-      <!-- Joint L4 - EL05 Motor 4 -->
+      <!-- Joint L4 - ${wrist_motor_type} Motor 4 -->
       <joint name="L4_joint">
         <param name="motor_id">4</param>
-        <param name="motor_type">EL05</param>
-        <param name="position_offset">0.0</param>
-        <param name="direction">1.0</param>
-        <command_interface name="position">
-          <param name="min">-1.5708</param>
-          <param name="max">1.5708</param>
-        </command_interface>
-        <command_interface name="velocity">
-          <param name="min">-50.0</param>
-          <param name="max">50.0</param>
-        </command_interface>
-        <command_interface name="effort">
-          <param name="min">-6.0</param>
-          <param name="max">6.0</param>
-        </command_interface>
-        <state_interface name="position"/>
-        <state_interface name="velocity"/>
-        <state_interface name="effort"/>
-      </joint>
-      <!-- Joint L5 - EL05 Motor 5 -->
+        <param name="motor_type">${wrist_motor_type}</param>
+        <param name="position_offset">0.0</param>
+        <param name="direction">1.0</param>
+        <param name="kp">30.0</param>
+        <param name="kd">2.0</param>
+        <command_interface name="position">
+          <param name="min">-1.5708</param>
+          <param name="max">1.5708</param>
+        </command_interface>
+        <command_interface name="velocity">
+          <param name="min">-50.0</param>
+          <param name="max">50.0</param>
+        </command_interface>
+        <command_interface name="effort">
+          <param name="min">${wrist_effort_min}</param>
+          <param name="max">${wrist_effort_max}</param>
+        </command_interface>
+        <state_interface name="position"/>
+        <state_interface name="velocity"/>
+        <state_interface name="effort"/>
+      </joint>
+      <!-- Joint L5 - ${wrist_motor_type} Motor 5 -->
       <joint name="L5_joint">
         <param name="motor_id">5</param>
-        <param name="motor_type">EL05</param>
+        <param name="motor_type">${wrist_motor_type}</param>
         <param name="position_offset">0.0</param>
         <param name="direction">-1.0</param>
-        <command_interface name="position">
-          <param name="min">-1.5708</param>
-          <param name="max">1.5708</param>
-        </command_interface>
-        <command_interface name="velocity">
-          <param name="min">-50.0</param>
-          <param name="max">50.0</param>
-        </command_interface>
-        <command_interface name="effort">
-          <param name="min">-6.0</param>
-          <param name="max">6.0</param>
-        </command_interface>
-        <state_interface name="position"/>
-        <state_interface name="velocity"/>
-        <state_interface name="effort"/>
-      </joint>
-      <!-- Joint L6 - EL05 Motor 6 -->
+        <param name="kp">30.0</param>
+        <param name="kd">2.0</param>
+        <command_interface name="position">
+          <param name="min">-1.5708</param>
+          <param name="max">1.5708</param>
+        </command_interface>
+        <command_interface name="velocity">
+          <param name="min">-50.0</param>
+          <param name="max">50.0</param>
+        </command_interface>
+        <command_interface name="effort">
+          <param name="min">${wrist_effort_min}</param>
+          <param name="max">${wrist_effort_max}</param>
+        </command_interface>
+        <state_interface name="position"/>
+        <state_interface name="velocity"/>
+        <state_interface name="effort"/>
+      </joint>
+      <!-- Joint L6 - ${wrist_motor_type} Motor 6 -->
       <joint name="L6_joint">
         <param name="motor_id">6</param>
-        <param name="motor_type">EL05</param>
-        <param name="position_offset">0.0</param>
-        <param name="direction">1.0</param>
-        <command_interface name="position">
-          <param name="min">-1.5708</param>
-          <param name="max">1.5708</param>
-        </command_interface>
-        <command_interface name="velocity">
-          <param name="min">-50.0</param>
-          <param name="max">50.0</param>
-        </command_interface>
-        <command_interface name="effort">
-          <param name="min">-6.0</param>
-          <param name="max">6.0</param>
+        <param name="motor_type">${wrist_motor_type}</param>
+        <param name="position_offset">0.0</param>
+        <param name="direction">1.0</param>
+        <param name="kp">30.0</param>
+        <param name="kd">2.0</param>
+        <command_interface name="position">
+          <param name="min">-1.5708</param>
+          <param name="max">1.5708</param>
+        </command_interface>
+        <command_interface name="velocity">
+          <param name="min">-50.0</param>
+          <param name="max">50.0</param>
+        </command_interface>
+        <command_interface name="effort">
+          <param name="min">${wrist_effort_min}</param>
+          <param name="max">${wrist_effort_max}</param>
+        </command_interface>
+        <state_interface name="position"/>
+        <state_interface name="velocity"/>
+        <state_interface name="effort"/>
+      </joint>
+      <!-- Joint L7 - ${wrist_motor_type} Motor 7 (Gripper) -->
+      <joint name="L7_joint">
+        <param name="motor_id">7</param>
+        <param name="motor_type">${wrist_motor_type}</param>
+        <param name="position_offset">0.0</param>
+        <param name="direction">1.0</param>
+        <command_interface name="position">
+          <param name="min">-1.5708</param>
+          <param name="max">1.5708</param>
+        </command_interface>
+        <command_interface name="velocity">
+          <param name="min">-50.0</param>
+          <param name="max">50.0</param>
+        </command_interface>
+        <command_interface name="effort">
+          <param name="min">${wrist_effort_min}</param>
+          <param name="max">${wrist_effort_max}</param>
         </command_interface>
         <state_interface name="position"/>
