Commit message: feat: SDK零力矩模式逐关节Kd、动力学标定边界修正、el_a3品牌统一
- 添加 dynamics_calibration.py 逐点增量保存标定脚本
- 修正 L6_com_z/L3_com_y/L5_mass 优化边界，提升标定精度 (RMSE 0.1037, R²=0.9925)
- ZeroTorqueModeWithGravity 支持逐关节 Kd 列表
- 固定质量标定模式 (--fix-masses)
- el_a3 品牌重命名及文档更新

Made-with: Cursor

File: el_a3_description/urdf/el_a3.urdf (robot description, URDF)
Before this commit: robot EL-A3, 9 links, 8 joints
Links:
- added link gripper_link, mass 0.05
- link l4_l5_urdf_asm: mass 0.44692 -> 0.54692
- link l5_l6_urdf_asm: mass 0.5317 -> 0.6317
Joints:
- added joint L7_joint: type revolute, parent l5_l6_urdf_asm, child gripper_link, origin xyz=0 0 -0.074 rpy=0 0 0, axis 0 0 1, limit lower=-1.5708 upper=1.5708 effort=6.0 velocity=50

File: el_a3_description/urdf/el_a3.urdf.xacro (robot description, xacro)
@@ -253,5 +253,5 @@
     <inertial>
       <origin xyz="-0.0241077 0.0297756 -0.000254349" rpy="0 0 0"/>
-      <mass value="0.44692"/>
+      <mass value="0.54692"/>
       <inertia ixx="0.000543249" ixy="0.000320527" ixz="2.88671e-06"
                iyy="0.00040341" iyz="-3.57587e-06" izz="0.000797799"/>
@@ -355,5 +355,5 @@
     <inertial>
       <origin xyz="-1.16996e-05 0.000627615 -0.0701883" rpy="0 0 0"/>
-      <mass value="0.5317"/>
+      <mass value="0.6317"/>
       <inertia ixx="0.00100405" ixy="-4.97095e-06" ixz="1.06714e-07"
                iyy="0.00139953" iyz="1.65952e-05" izz="0.00054217"/>

File: el_a3_description/urdf/el_a3_ros2_control.xacro (robot description, xacro)
@@ -16,6 +16,6 @@
           <param name="can_interface">${can_interface}</param>
           <param name="host_can_id">${host_can_id}</param>
-          <param name="position_kp">55.0</param>
-          <param name="position_kd">4.5</param>
+          <param name="position_kp">100.0</param>
+          <param name="position_kd">4.0</param>
           <param name="velocity_limit">10.0</param>
           <!-- S-curve trajectory planning parameters -->
@@ -27,13 +27,12 @@
           <param name="smoothing_alpha">0.8</param>     <!-- Low-pass filter coefficient (0.8 = near-passthrough, teleop already smooths) -->
           <!-- Gravity compensation feedforward parameters (100% gravity as feedforward torque, matching zero-torque mode) -->
-          <param name="gravity_feedforward_ratio">0.85</param>  <!-- 85% gravity compensation ratio, avoid over-compensation oscillation -->
+          <param name="gravity_feedforward_ratio">0.0</param>  <!-- Gravity feedforward disabled -->
           <!-- Zero-torque mode parameters -->
           <param name="zero_torque_kd">0.3</param>  <!-- Zero-torque mode damping coefficient -->
           <!-- Pinocchio dynamics model configuration -->
-          <!-- Note: Requires absolute path to URDF file -->
-          <param name="urdf_path">/home/wy/RS/A3/el_a3_description/urdf/el_a3.urdf</param>
+          <param name="urdf_path">$(find el_a3_description)/urdf/el_a3.urdf</param>
           <param name="use_pinocchio_gravity">true</param>  <!-- Enable full dynamics gravity compensation -->
           <!-- Inertia parameter config file path (generated by inertia_calibration.py) -->
-          <param name="inertia_config_path">/home/wy/RS/A3/el_a3_description/config/inertia_params.yaml</param>
+          <param name="inertia_config_path">$(find el_a3_description)/config/inertia_params.yaml</param>
           <!-- Inertia parameter scale factors (legacy method, kept for backward compatibility) -->
           <param name="inertia_scale_L1_mass">1.0000</param>
@@ -142,6 +141,6 @@
         <param name="position_offset">0.0</param>
         <param name="direction">1.0</param>
-        <param name="kp">30.0</param>
-        <param name="kd">2.0</param>
+        <param name="kp">100.0</param>
+        <param name="kd">4.0</param>
         <command_interface name="position">
           <param name="min">-1.5708</param>
@@ -166,6 +165,6 @@
         <param name="position_offset">0.0</param>
         <param name="direction">-1.0</param>
-        <param name="kp">30.0</param>
-        <param name="kd">2.0</param>
+        <param name="kp">100.0</param>
+        <param name="kd">4.0</param>
         <command_interface name="position">
           <param name="min">-1.5708</param>
@@ -190,6 +189,6 @@
         <param name="position_offset">0.0</param>
         <param name="direction">1.0</param>
-        <param name="kp">30.0</param>
-        <param name="kd">2.0</param>
+        <param name="kp">100.0</param>
+        <param name="kd">4.0</param>
         <command_interface name="position">
           <param name="min">-1.5708</param>

File: ros2_ws/src/el_a3_web_ui/static/urdf/el_a3.urdf (robot description, URDF)
Before this commit: robot EL-A3, 9 links, 8 joints
Links:
- added link gripper_link, mass 0.05
- link l4_l5_urdf_asm: mass 0.44692 -> 0.54692
- link l5_l6_urdf_asm: mass 0.5317 -> 0.6317
Joints:
- added joint L7_joint: type revolute, parent l5_l6_urdf_asm, child gripper_link, origin xyz=0 0 -0.074 rpy=0 0 0, axis 0 0 1, limit lower=-1.5708 upper=1.5708 effort=6.0 velocity=50
